File: hardware/ctrl-v0.1/icetwang-controller.kicad_pcb (KiCad board)
At the start: 2 copper layers, 38 x 61 mm, 52 parts, among them J1 IMU STEMMA QT, J10 SPKR_PWR, J2 IMU SPI, J3 JOY, J4 SPKR AMP, J5 OLED, J6 RGB_LED, J7 RJ45, J8 POLE5V, J9 POLEGND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

Commit message: Swapped to NULL logos and added pdf schematics.
Parts:
- REF**: value 1b2_Logo_SilkS_6mm -> null_Logo_SilkS_6mm; footprint pkl_logos:1b2_Logo_SilkS_6mm -> pkl_logos:null_Logo_SilkS_6mm
- REF**: value 1b2_Logo_SilkS_10mm -> null_Logo_SilkS_10mm; footprint pkl_logos:1b2_Logo_SilkS_10mm -> pkl_logos:null_Logo_SilkS_10mm
Other:
- board text added: "NULL"
- board text added: "iCE-TWANG Controller V0.1 CC-BY-SA"
- board text removed: "1BitSquared"
Changed lines of the file:
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@@
     )
   )
-  (footprint "pkl_logos:1b2_Logo_SilkS_6mm" (layer "F.Cu")
+  (footprint "pkl_logos:null_Logo_SilkS_6mm" (layer "F.Cu")
     (at 24.9 29.9)
-    (descr "1BitSquared Logo, Silk Screen, 6mm")
-    (tags "logo symbol 1bitsquared 1b2")
+    (descr "NULL Logo, Silk Screen, 6mm")
+    (tags "logo symbol null")
     (attr exclude_from_pos_files exclude_from_bom)
     (fp_text reference "REF**" (at 0 -4) (layer "F.SilkS") hide
       (effects (font (size 1 1) (thickness 0.15)))
     )
-    (fp_text value "1b2_Logo_SilkS_6mm" (at 0 4) (layer "F.Fab") hide
-      (effects (font (size 1 1) (thickness 0.15)))
-    )
-    (fp_line (start -0.6 -0.6) (end -3 -0.6) (layer "F.SilkS") (width 0.24))
-    (fp_line (start -3 -0.6) (end -3 -3) (layer "F.SilkS") (width 0.24))
-    (fp_line (start 0 -2.4) (end 0 0) (layer "F.SilkS") (width 0.24))
-    (fp_line (start 2.4 -2.4) (end 2.4 2.4) (layer "F.SilkS") (width 0.24))
-    (fp_line (start 3 3) (end -1.8 3) (layer "F.SilkS") (width 0.24))
-    (fp_line (start 3 -1.8) (end 3 3) (layer "F.SilkS") (width 0.24))
-    (fp_line (start -3 -3) (end -0.6 -3) (layer "F.SilkS") (width 0.24))
-    (fp_line (start -0.6 -3) (end 0 -2.4) (layer "F.SilkS") (width 0.24))
-    (fp_line (start 0.6 -2.4) (end 2.4 -2.4) (layer "F.SilkS") (width 0.24))
-    (fp_line (start 2.4 2.4) (end 3 3) (layer "F.SilkS") (width 0.24))
-    (fp_line (start -2.4 2.4) (end -2.4 0.6) (layer "F.SilkS") (width 0.24))
-    (fp_line (start -1.8 3) (end -2.4 2.4) (layer "F.SilkS") (width 0.24))
-    (fp_line (start 2.4 -2.4) (end 3 -1.8) (layer "F.SilkS") (width 0.24))
-    (fp_line (start 0 0) (end -2.4 0) (layer "F.SilkS") (width 0.24))
-    (fp_line (start -0.6 -0.6) (end 0 0) (layer "F.SilkS") (width 0.24))
-    (fp_line (start 0.6 0.6) (end 0.6 -2.4) (layer "F.SilkS") (width 0.24))
-    (fp_line (start -2.4 0.6) (end 0.6 0.6) (layer "F.SilkS") (width 0.24))
-    (fp_line (start 2.4 2.4) (end -2.4 2.4) (layer "F.SilkS") (width 0.24))
-    (fp_line (start -0.6 -3) (end -0.6 -0.6) (layer "F.SilkS") (width 0.24))
-    (fp_line (start -2.4 0) (end -3 -0.6) (layer "F.SilkS") (width 0.24))
+    (fp_text value "null_Logo_SilkS_6mm" (at 0 4) (layer "F.Fab") hide
+      (effects (font (size 1 1) (thickness 0.15)))
+    )
+    (fp_line (start -1.5 -0.5) (end -1 0.5) (layer "F.SilkS") (width 0.15))
+    (fp_line (start 0.2 0.5) (end 0.7 0.5) (layer "F.SilkS") (width 0.15))
+    (fp_line (start 0.2 -0.5) (end 0.2 0.5) (layer "F.SilkS") (width 0.15))
+    (fp_line (start 3 -3) (end 3 3) (layer "F.SilkS") (width 0.24))
+    (fp_line (start -3 -3) (end -3 3) (layer "F.SilkS") (width 0.24))
+    (fp_line (start -0.1 0.2) (end -0.1 -0.5) (layer "F.SilkS") (width 0.15))
+    (fp_line (start -0.7 -0.5) (end -0.7 0.2) (layer "F.SilkS") (width 0.15))
+    (fp_line (start -1.5 0.5) (end -1.5 -0.5) (layer "F.SilkS") (width 0.15))
+    (fp_line (start 3 -3) (end -3 -3) (layer "F.SilkS") (width 0.24))
+    (fp_line (start 1 -0.5) (end 1 0.5) (layer "F.SilkS") (width 0.15))
+    (fp_line (start -1 0.5) (end -1 -0.5) (layer "F.SilkS") (width 0.15))
+    (fp_line (start 1 0.5) (end 1.5 0.5) (layer "F.SilkS") (width 0.15))
+    (fp_line (start -3 3) (end 3 3) (layer "F.SilkS") (width 0.24))
+    (fp_arc (start -0.4 0.2) (end -0.7 0.2) (angle -180) (layer "F.SilkS") (width 0.15))
   )
   (footprint "Connector_Molex:Molex_PicoBlade_53261-0771_1x07-1MP_P1.25mm_Horizontal" (layer "F.Cu")
@@
       (net 33 "/POLEGND") (pintype "passive"))
   )
-  (footprint "pkl_logos:1b2_Logo_SilkS_10mm" (layer "B.Cu")
+  (footprint "pkl_logos:null_Logo_SilkS_10mm" (layer "B.Cu")
     (at 44 54.8 180)
-    (descr "1BitSquared Logo, Silk Screen, 10mm")
-    (tags "logo symbol 1bitsquared 1b2")
+    (descr "NULL Logo, Silk Screen, 10mm")
+    (tags "logo symbol null")
     (attr exclude_from_pos_files exclude_from_bom)
     (fp_text reference "REF**" (at 0 6) (layer "B.SilkS") hide
       (effects (font (size 1 1) (thickness 0.15)) (justify mirror))
     )
-    (fp_text value "1b2_Logo_SilkS_10mm" (at 0 -6) (layer "B.Fab") hide
+    (fp_text value "null_Logo_SilkS_10mm" (at 0 -6) (layer "B.Fab") hide
       (effects (font (size 1 1) (thickness 0.15)) (justify mirror))
     )
-    (fp_line (start 0 4) (end 0 0) (layer "B.SilkS") (width 0.4))
-    (fp_line (start 4 4) (end 1 4) (layer "B.SilkS") (width 0.4))
-    (fp_line (start -1 5) (end 0 4) (layer "B.SilkS") (width 0.4))
-    (fp_line (start -1 5) (end -5 5) (layer "B.SilkS") (width 0.4))
-    (fp_line (start -5 5) (end -5 1) (layer "B.SilkS") (width 0.4))
-    (fp_line (start 4 4) (end 5 3) (layer "B.SilkS") (width 0.4))
-    (fp_line (start -5 1) (end -1 1) (layer "B.SilkS") (width 0.4))
-    (fp_line (start 1 4) (end 1 -1) (layer "B.SilkS") (width 0.4))
-    (fp_line (start -4 -4) (end -3 -5) (layer "B.SilkS") (width 0.4))
-    (fp_line (start -3 -5) (end 5 -5) (layer "B.SilkS") (width 0.4))
-    (fp_line (start 1 -1) (end -4 -1) (layer "B.SilkS") (width 0.4))
-    (fp_line (start -4 0) (end 0 0) (layer "B.SilkS") (width 0.4))
-    (fp_line (start -4 -4) (end 4 -4) (layer "B.SilkS") (width 0.4))
-    (fp_line (start 5 -5) (end 4 -4) (layer "B.SilkS") (width 0.4))
-    (fp_line (start -1 1) (end -1 5) (layer "B.SilkS") (width 0.4))
-    (fp_line (start -4 -1) (end -4 -4) (layer "B.SilkS") (width 0.4))
-    (fp_line (start 5 3) (end 5 -5) (layer "B.SilkS") (width 0.4))
-    (fp_line (start -5 1) (end -4 0) (layer "B.SilkS") (width 0.4))
-    (fp_line (start 0 0) (end -1 1) (layer "B.SilkS") (width 0.4))
-    (fp_line (start 4 -4) (end 4 4) (layer "B.SilkS") (width 0.4))
+    (fp_line (start 0.2 0.5) (end 0.2 -0.5) (layer "B.SilkS") (width 0.15))
+    (fp_line (start -1 -0.5) (end -1 0.5) (layer "B.SilkS") (width 0.15))
+    (fp_line (start 0.2 -0.5) (end 0.7 -0.5) (layer "B.SilkS") (width 0.15))
+    (fp_line (start -0.7 0.5) (end -0.7 -0.2) (layer "B.SilkS") (width 0.15))
+    (fp_line (start 5 5) (end 5 -5) (layer "B.SilkS") (width 0.4))
+    (fp_line (start -1.5 0.5) (end -1 -0.5) (layer "B.SilkS") (width 0.15))
+    (fp_line (start -5 5) (end -5 -5) (layer "B.SilkS") (width 0.4))
+    (fp_line (start 1 -0.5) (end 1.5 -0.5) (layer "B.SilkS") (width 0.15))
+    (fp_line (start 5 5) (end -5 5) (layer "B.SilkS") (width 0.4))
+    (fp_line (start -1.5 -0.5) (end -1.5 0.5) (layer "B.SilkS") (width 0.15))
+    (fp_line (start -5 -5) (end 5 -5) (layer "B.SilkS") (width 0.4))
+    (fp_line (start 1 0.5) (end 1 -0.5) (layer "B.SilkS") (width 0.15))
+    (fp_line (start -0.1 0.5) (end -0.1 -0.2) (layer "B.SilkS") (width 0.15))
+    (fp_arc (start -0.4 -0.2) (end -0.7 -0.2) (angle 180) (layer "B.SilkS") (width 0.15))
   )
   (footprint "pkl_jumpers:J_NC_0603_40" (layer "B.Cu")
@@
     (effects (font (size 1.5 1.5) (thickness 0.3)) (justify mirror))
   )
-  (gr_text "1BitSquared" (at 43.5 61.4) (layer "B.SilkS")
+  (gr_text "NULL" (at 43.5 61.4) (layer "B.SilkS")
     (effects (font (size 1.5 1.5) (thickness 0.3)) (justify mirror))
   )
@@
     (effects (font (size 1 1) (thickness 0.15)))
   )
-  (gr_text "iCE-TWANG\nController\nV0.1" (at 25.2 42.3) (layer "F.SilkS")
+  (gr_text "iCE-TWANG\nController\nV0.1\nCC-BY-SA" (at 25.2 41.6) (layer "F.SilkS")
     (effects (font (size 1 1) (thickness 0.15)))
   )
@@
     (effects (font (size 1 1) (thickness 0.15)))
   )
-  (gr_text "1BitSquared" (at 25.2 34) (layer "F.SilkS")
+  (gr_text "NULL" (at 25.2 34) (layer "F.SilkS")
     (effects (font (size 1 1) (thickness 0.15)))
   )
